Commit message: update api for loading urdf models

File: src/gym_gz_models/iCubGazeboSimpleCollisionsV2_5/icub_simple_collisions.urdf (robot description, URDF)
Before this commit: robot iCubGazeboSimpleCollisionsV2_5, 52 links, 51 joints
Links:
- link chest: geometry collision box size=0.15 0.18 0.26; visual mesh filename=package://meshes/simmechanics/sim_sea_2-5_chest_bb_prt-bina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 scale=0.001 0.001 0.001
- link head: geometry collision sphere radius=0.11; visual mesh filename=package://meshes/simmechanics/sim_sea_2-5_head_prt-binary.s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 scale=0.001 0.001 0.001
- link l_ankle_1: geometry visual mesh filename=package://meshes/simmechanics/sim_sea_2-5_l_ankle_prt-binar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 scale=0.001 0.001 0.001
- link l_ankle_2: geometry visual mesh filename=package://meshes/simmechanics/sim_sea_2-5_l_foot_prt-binary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 scale=0.001 0.001 0.001
- link l_elbow_1: geometry visual mesh filename=package://meshes/simmechanics/sim_sea_2-5_l_elbow_prosup_pr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 scale=0.001 0.001 0.001
- link l_foot: geometry collision box size=0.16 0.072 0.001; visual mesh filename=package://meshes/simmechanics/sim_sea_2-5_l_sole_prt-binary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 scale=0.001 0.001 0.001
- link l_forearm: geometry collision cylinder length=0.12 radius=0.04; visual mesh filename=package://meshes/simmechanics/sim_sea_2-5_l_forearm_prt-bin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 scale=0.001 0.001 0.001
- link l_hand: geometry collision box size=0.14 0.05 0.07; visual mesh filename=package://meshes/simmechanics/sim_sea_2-5_l_hand_prt-binary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 scale=0.001 0.001 0.001
- link l_hip_1: geometry visual mesh filename=package://meshes/simmechanics/sim_sea_2-5_l_hip_1_prt-binar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 scale=0.001 0.001 0.001
- link l_hip_2: geometry visual mesh filename=package://meshes/simmechanics/sim_sea_2-5_l_hip_2_prt-binar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 scale=0.001 0.001 0.001
- link l_hip_3: geometry visual mesh filename=package://meshes/simmechanics/sim_sea_2-5_l_upper_thigh_prt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 scale=0.001 0.001 0.001
- link l_lower_leg: geometry collision cylinder length=0.20 radius=0.056; visual mesh filename=package://meshes/simmechanics/sim_sea_2-5_l_shank_prt-binar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 scale=0.001 0.001 0.001
- link l_shoulder_1: geometry visual mesh filename=package://meshes/simmechanics/sim_sea_2-5_l_shoulder_1_prt-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 scale=0.001 0.001 0.001
- link l_shoulder_2: geometry visual mesh filename=package://meshes/simmechanics/sim_sea_2-5_l_shoulder_2_prt-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 scale=0.001 0.001 0.001
- link l_shoulder_3: geometry visual mesh filename=package://meshes/simmechanics/sim_sea_2-5_l_upper_arm_prt-b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 scale=0.001 0.001 0.001
- link l_upper_arm: geometry collision cylinder length=0.13 radius=0.047; visual mesh filename=package://meshes/simmechanics/sim_sea_2-5_l_elbow_prt-binar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 scale=0.001 0.001 0.001
- link l_upper_leg: geometry collision cylinder length=0.16 radius=0.06; visual mesh filename=package://meshes/simmechanics/sim_sea_2-5_l_thigh_prt-binar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 scale=0.001 0.001 0.001
- link l_wrist_1: geometry visual mesh filename=package://meshes/simmechanics/sim_sea_2-5_l_wrist_pitch_prt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 scale=0.001 0.001 0.001
- link neck_1: geometry visual mesh filename=package://meshes/simmechanics/sim_sea_2-5_neck_1_prt-binary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 scale=0.001 0.001 0.001
- link neck_2: geometry visual mesh filename=package://meshes/simmechanics/sim_sea_2-5_neck_2_prt-binary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 scale=0.001 0.001 0.001
- link r_ankle_1: geometry visual mesh filename=package://meshes/simmechanics/sim_sea_2-5_r_ankle_prt-binar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 scale=0.001 0.001 0.001
- link r_ankle_2: geometry visual mesh filename=package://meshes/simmechanics/sim_sea_2-5_r_foot_prt-binary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 scale=0.001 0.001 0.001
- link r_elbow_1: geometry visual mesh filename=package://meshes/simmechanics/sim_sea_2-5_r_elbow_prosup_pr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 scale=0.001 0.001 0.001
- link r_foot: geometry collision box size=0.16 0.072 0.001; visual mesh filename=package://meshes/simmechanics/sim_sea_2-5_r_sole_prt-binary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 scale=0.001 0.001 0.001
- link r_forearm: geometry collision cylinder length=0.12 radius=0.04; visual mesh filename=package://meshes/simmechanics/sim_sea_2-5_r_forearm_prt-bin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 scale=0.001 0.001 0.001
- link r_hand: geometry collision box size=0.14 0.05 0.07; visual mesh filename=package://meshes/simmechanics/sim_sea_2-5_r_hand_prt-binary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 scale=0.001 0.001 0.001
- link r_hip_1: geometry visual mesh filename=package://meshes/simmechanics/sim_sea_2-5_r_hip_1_prt-binar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 scale=0.001 0.001 0.001
- link r_hip_2: geometry visual mesh filename=package://meshes/simmechanics/sim_sea_2-5_r_hip_2_prt-binar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 scale=0.001 0.001 0.001
- link r_hip_3: geometry visual mesh filename=package://meshes/simmechanics/sim_sea_2-5_r_upper_thigh_prt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 scale=0.001 0.001 0.001
- link r_lower_leg: geometry collision cylinder length=0.20 radius=0.056; visual mesh filename=package://meshes/simmechanics/sim_sea_2-5_r_shank_prt-binar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 scale=0.001 0.001 0.001
- link r_shoulder_1: geometry visual mesh filename=package://meshes/simmechanics/sim_sea_2-5_r_shoulder_1_prt-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 scale=0.001 0.001 0.001
- link r_shoulder_2: geometry visual mesh filename=package://meshes/simmechanics/sim_sea_2-5_r_shoulder_2_prt-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 scale=0.001 0.001 0.001
- link r_shoulder_3: geometry visual mesh filename=package://meshes/simmechanics/sim_sea_2-5_r_upper_arm_prt-b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 scale=0.001 0.001 0.001
- link r_upper_arm: geometry collision cylinder length=0.13 radius=0.047; visual mesh filename=package://meshes/simmechanics/sim_sea_2-5_r_elbow_prt-binar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 scale=0.001 0.001 0.001
- link r_upper_leg: geometry collision cylinder length=0.16 radius=0.06; visual mesh filename=package://meshes/simmechanics/sim_sea_2-5_r_thigh_prt-binar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 scale=0.001 0.001 0.001
- link r_wrist_1: geometry visual mesh filename=package://meshes/simmechanics/sim_sea_2-5_r_wrist_pitch_prt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 scale=0.001 0.001 0.001
- link root_link: geometry collision box size=0.13 0.2 0.13; visual mesh filename=package://meshes/simmechanics/sim_sea_2-5_root_link_prt-bin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 scale=0.001 0.001 0.001
- link torso_1: geometry visual mesh filename=package://meshes/simmechanics/sim_sea_2-5_lap_belt_1_prt-bi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 scale=0.001 0.001 0.001
- link torso_2: geometry visual mesh filename=package://meshes/simmechanics/sim_sea_2-5_lap_belt_2_prt-bi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 scale=0.001 0.001 0.001

File: src/gym_gz_models/iCubGazeboV2_5/icub.urdf (robot description, URDF)
Before this commit: robot iCubGazeboV2_5, 52 links, 51 joints
Links:
- link chest: geometry collision mesh filename=package://meshes/simmechanics/sim_sea_2-5_chest_bb_prt-bina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 scale=0.001 0.001 0.001; visual mesh filename=package://meshes/simmechanics/sim_sea_2-5_chest_bb_prt-bina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 scale=0.001 0.001 0.001
- link head: geometry collision mesh filename=package://meshes/simmechanics/sim_sea_2-5_head_prt-binary.s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 scale=0.001 0.001 0.001; visual mesh filename=package://meshes/simmechanics/sim_sea_2-5_head_prt-binary.s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 scale=0.001 0.001 0.001
- link l_ankle_1: geometry collision mesh filename=package://meshes/simmechanics/sim_sea_2-5_l_ankle_prt-binar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 scale=0.001 0.001 0.001; visual mesh filename=package://meshes/simmechanics/sim_sea_2-5_l_ankle_prt-binar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 scale=0.001 0.001 0.001
- link l_ankle_2: geometry collision mesh filename=package://meshes/simmechanics/sim_sea_2-5_l_foot_prt-binary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 scale=0.001 0.001 0.001; visual mesh filename=package://meshes/simmechanics/sim_sea_2-5_l_foot_prt-binary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 scale=0.001 0.001 0.001
- link l_elbow_1: geometry collision mesh filename=package://meshes/simmechanics/sim_sea_2-5_l_elbow_prosup_pr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 scale=0.001 0.001 0.001; visual mesh filename=package://meshes/simmechanics/sim_sea_2-5_l_elbow_prosup_pr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 scale=0.001 0.001 0.001
- link l_foot: geometry collision box size=0.16 0.072 0.001; visual mesh filename=package://meshes/simmechanics/sim_sea_2-5_l_sole_prt-binary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 scale=0.001 0.001 0.001
- link l_forearm: geometry collision mesh filename=package://meshes/simmechanics/sim_sea_2-5_l_forearm_prt-bin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 scale=0.001 0.001 0.001; visual mesh filename=package://meshes/simmechanics/sim_sea_2-5_l_forearm_prt-bin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 scale=0.001 0.001 0.001
- link l_hand: geometry collision mesh filename=package://meshes/simmechanics/sim_sea_2-5_l_hand_prt-binary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 scale=0.001 0.001 0.001; visual mesh filename=package://meshes/simmechanics/sim_sea_2-5_l_hand_prt-binary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 scale=0.001 0.001 0.001
- link l_hip_1: geometry collision mesh filename=package://meshes/simmechanics/sim_sea_2-5_l_hip_1_prt-binar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 scale=0.001 0.001 0.001; visual mesh filename=package://meshes/simmechanics/sim_sea_2-5_l_hip_1_prt-binar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 scale=0.001 0.001 0.001
- link l_hip_2: geometry collision mesh filename=package://meshes/simmechanics/sim_sea_2-5_l_hip_2_prt-binar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 scale=0.001 0.001 0.001; visual mesh filename=package://meshes/simmechanics/sim_sea_2-5_l_hip_2_prt-binar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 scale=0.001 0.001 0.001
- link l_hip_3: geometry collision mesh filename=package://meshes/simmechanics/sim_sea_2-5_l_upper_thigh_prt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 scale=0.001 0.001 0.001; visual mesh filename=package://meshes/simmechanics/sim_sea_2-5_l_upper_thigh_prt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 scale=0.001 0.001 0.001
- link l_lower_leg: geometry collision mesh filename=package://meshes/simmechanics/sim_sea_2-5_l_shank_prt-binar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 scale=0.001 0.001 0.001; visual mesh filename=package://meshes/simmechanics/sim_sea_2-5_l_shank_prt-binar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 scale=0.001 0.001 0.001
- link l_shoulder_1: geometry collision mesh filename=package://meshes/simmechanics/sim_sea_2-5_l_shoulder_1_prt-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 scale=0.001 0.001 0.001; visual mesh filename=package://meshes/simmechanics/sim_sea_2-5_l_shoulder_1_prt-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 scale=0.001 0.001 0.001
- link l_shoulder_2: geometry collision mesh filename=package://meshes/simmechanics/sim_sea_2-5_l_shoulder_2_prt-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 scale=0.001 0.001 0.001; visual mesh filename=package://meshes/simmechanics/sim_sea_2-5_l_shoulder_2_prt-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 scale=0.001 0.001 0.001
- link l_shoulder_3: geometry collision mesh filename=package://meshes/simmechanics/sim_sea_2-5_l_upper_arm_prt-b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 scale=0.001 0.001 0.001; visual mesh filename=package://meshes/simmechanics/sim_sea_2-5_l_upper_arm_prt-b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 scale=0.001 0.001 0.001
- link l_upper_arm: geometry collision mesh filename=package://meshes/simmechanics/sim_sea_2-5_l_elbow_prt-binar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 scale=0.001 0.001 0.001; visual mesh filename=package://meshes/simmechanics/sim_sea_2-5_l_elbow_prt-binar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 scale=0.001 0.001 0.001
- link l_upper_leg: geometry collision mesh filename=package://meshes/simmechanics/sim_sea_2-5_l_thigh_prt-binar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 scale=0.001 0.001 0.001; visual mesh filename=package://meshes/simmechanics/sim_sea_2-5_l_thigh_prt-binar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 scale=0.001 0.001 0.001
- link l_wrist_1: geometry collision mesh filename=package://meshes/simmechanics/sim_sea_2-5_l_wrist_pitch_prt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 scale=0.001 0.001 0.001; visual mesh filename=package://meshes/simmechanics/sim_sea_2-5_l_wrist_pitch_prt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 scale=0.001 0.001 0.001
- link neck_1: geometry collision mesh filename=package://meshes/simmechanics/sim_sea_2-5_neck_1_prt-binary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 scale=0.001 0.001 0.001; visual mesh filename=package://meshes/simmechanics/sim_sea_2-5_neck_1_prt-binary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 scale=0.001 0.001 0.001
- link neck_2: geometry collision mesh filename=package://meshes/simmechanics/sim_sea_2-5_neck_2_prt-binary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 scale=0.001 0.001 0.001; visual mesh filename=package://meshes/simmechanics/sim_sea_2-5_neck_2_prt-binary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 scale=0.001 0.001 0.001
- link r_ankle_1: geometry collision mesh filename=package://meshes/simmechanics/sim_sea_2-5_r_ankle_prt-binar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 scale=0.001 0.001 0.001; visual mesh filename=package://meshes/simmechanics/sim_sea_2-5_r_ankle_prt-binar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 scale=0.001 0.001 0.001
- link r_ankle_2: geometry collision mesh filename=package://meshes/simmechanics/sim_sea_2-5_r_foot_prt-binary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 scale=0.001 0.001 0.001; visual mesh filename=package://meshes/simmechanics/sim_sea_2-5_r_foot_prt-binary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 scale=0.001 0.001 0.001
- link r_elbow_1: geometry collision mesh filename=package://meshes/simmechanics/sim_sea_2-5_r_elbow_prosup_pr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 scale=0.001 0.001 0.001; visual mesh filename=package://meshes/simmechanics/sim_sea_2-5_r_elbow_prosup_pr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 scale=0.001 0.001 0.001
- link r_foot: geometry collision box size=0.16 0.072 0.001; visual mesh filename=package://meshes/simmechanics/sim_sea_2-5_r_sole_prt-binary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 scale=0.001 0.001 0.001
- link r_forearm: geometry collision mesh filename=package://meshes/simmechanics/sim_sea_2-5_r_forearm_prt-bin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 scale=0.001 0.001 0.001; visual mesh filename=package://meshes/simmechanics/sim_sea_2-5_r_forearm_prt-bin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 scale=0.001 0.001 0.001
- link r_hand: geometry collision mesh filename=package://meshes/simmechanics/sim_sea_2-5_r_hand_prt-binary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 scale=0.001 0.001 0.001; visual mesh filename=package://meshes/simmechanics/sim_sea_2-5_r_hand_prt-binary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 scale=0.001 0.001 0.001
- link r_hip_1: geometry collision mesh filename=package://meshes/simmechanics/sim_sea_2-5_r_hip_1_prt-binar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 scale=0.001 0.001 0.001; visual mesh filename=package://meshes/simmechanics/sim_sea_2-5_r_hip_1_prt-binar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 scale=0.001 0.001 0.001
- link r_hip_2: geometry collision mesh filename=package://meshes/simmechanics/sim_sea_2-5_r_hip_2_prt-binar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 scale=0.001 0.001 0.001; visual mesh filename=package://meshes/simmechanics/sim_sea_2-5_r_hip_2_prt-binar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 scale=0.001 0.001 0.001
- link r_hip_3: geometry collision mesh filename=package://meshes/simmechanics/sim_sea_2-5_r_upper_thigh_prt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 scale=0.001 0.001 0.001; visual mesh filename=package://meshes/simmechanics/sim_sea_2-5_r_upper_thigh_prt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 scale=0.001 0.001 0.001
- link r_lower_leg: geometry collision mesh filename=package://meshes/simmechanics/sim_sea_2-5_r_shank_prt-binar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 scale=0.001 0.001 0.001; visual mesh filename=package://meshes/simmechanics/sim_sea_2-5_r_shank_prt-binar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 scale=0.001 0.001 0.001
- link r_shoulder_1: geometry collision mesh filename=package://meshes/simmechanics/sim_sea_2-5_r_shoulder_1_prt-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 scale=0.001 0.001 0.001; visual mesh filename=package://meshes/simmechanics/sim_sea_2-5_r_shoulder_1_prt-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 scale=0.001 0.001 0.001
- link r_shoulder_2: geometry collision mesh filename=package://meshes/simmechanics/sim_sea_2-5_r_shoulder_2_prt-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 scale=0.001 0.001 0.001; visual mesh filename=package://meshes/simmechanics/sim_sea_2-5_r_shoulder_2_prt-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 scale=0.001 0.001 0.001
- link r_shoulder_3: geometry collision mesh filename=package://meshes/simmechanics/sim_sea_2-5_r_upper_arm_prt-b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 scale=0.001 0.001 0.001; visual mesh filename=package://meshes/simmechanics/sim_sea_2-5_r_upper_arm_prt-b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 scale=0.001 0.001 0.001
- link r_upper_arm: geometry collision mesh filename=package://meshes/simmechanics/sim_sea_2-5_r_elbow_prt-binar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 scale=0.001 0.001 0.001; visual mesh filename=package://meshes/simmechanics/sim_sea_2-5_r_elbow_prt-binar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 scale=0.001 0.001 0.001
- link r_upper_leg: geometry collision mesh filename=package://meshes/simmechanics/sim_sea_2-5_r_thigh_prt-binar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 scale=0.001 0.001 0.001; visual mesh filename=package://meshes/simmechanics/sim_sea_2-5_r_thigh_prt-binar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 scale=0.001 0.001 0.001
- link r_wrist_1: geometry collision mesh filename=package://meshes/simmechanics/sim_sea_2-5_r_wrist_pitch_prt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 scale=0.001 0.001 0.001; visual mesh filename=package://meshes/simmechanics/sim_sea_2-5_r_wrist_pitch_prt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 scale=0.001 0.001 0.001
- link root_link: geometry collision mesh filename=package://meshes/simmechanics/sim_sea_2-5_root_link_prt-bin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 scale=0.001 0.001 0.001; visual mesh filename=package://meshes/simmechanics/sim_sea_2-5_root_link_prt-bin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 scale=0.001 0.001 0.001
- link torso_1: geometry collision mesh filename=package://meshes/simmechanics/sim_sea_2-5_lap_belt_1_prt-bi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 scale=0.001 0.001 0.001; visual mesh filename=package://meshes/simmechanics/sim_sea_2-5_lap_belt_1_prt-bi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 scale=0.001 0.001 0.001
- link torso_2: geometry collision mesh filename=package://meshes/simmechanics/sim_sea_2-5_lap_belt_2_prt-bi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 scale=0.001 0.001 0.001; visual mesh filename=package://meshes/simmechanics/sim_sea_2-5_lap_belt_2_prt-bi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 scale=0.001 0.001 0.001

File: src/gym_gz_models/panda/panda.urdf (robot description, URDF)
Before this commit: robot panda, 14 links, 13 joints
Links:
- link panda_hand: geometry collision mesh filename=package://panda/meshes/collision/hand.stl; visual mesh filename=package://panda/meshes/visual/hand.dae
- link panda_leftfinger: geometry collision mesh filename=package://panda/meshes/collision/finger.stl; visual mesh filename=package://panda/meshes/visual/finger.dae
- link panda_link0: geometry collision mesh filename=package://panda/meshes/collision/link0.stl; visual mesh filename=package://panda/meshes/visual/link0.dae
- link panda_link1: geometry collision mesh filename=package://panda/meshes/collision/link1.stl; visual mesh filename=package://panda/meshes/visual/link1.dae
- link panda_link2: geometry collision mesh filename=package://panda/meshes/collision/link2.stl; visual mesh filename=package://panda/meshes/visual/link2.dae
- link panda_link3: geometry collision mesh filename=package://panda/meshes/collision/link3.stl; visual mesh filename=package://panda/meshes/visual/link3.dae
- link panda_link4: geometry collision mesh filename=package://panda/meshes/collision/link4.stl; visual mesh filename=package://panda/meshes/visual/link4.dae
- link panda_link5: geometry collision mesh filename=package://panda/meshes/collision/link5.stl; visual mesh filename=package://panda/meshes/visual/link5.dae
- link panda_link6: geometry collision mesh filename=package://panda/meshes/collision/link6.stl; visual mesh filename=package://panda/meshes/visual/link6.dae
- link panda_link7: geometry collision mesh filename=package://panda/meshes/collision/link7.stl; visual mesh filename=package://panda/meshes/visual/link7.dae
- link panda_rightfinger: geometry collision mesh filename=package://panda/meshes/collision/finger.stl; visual mesh filename=package://panda/meshes/visual/finger.dae
